File: hardware/kicad/hauptplatine/versorgung.kicad_sch (KiCad schematic)
At the start: 32 parts, among them J201 Solar 1, J202 Solar 2, J203 Akku (JST PH 4), U201 BQ25185DLHR, U202 RT9080-33GJ5, U203 TPS22917DBV

Commit message: test
Parts:
- added C212: 2,2µ, Capacitor_SMD:C_0603_1608Metric, symbol Device:C
- added U204: TPS70933DBV, Package_TO_SOT_SMD:SOT-23-5, symbol Bienen:TPS70933DBV
- C201: value 4,7µ 25V -> 4,7µ 50V X7R
- J203: value Akku (JST PH 4) -> Akku (JST PH 5); footprint Connector_JST:JST_PH_B4B-PH-K_1x04_P2.00mm_Vertical -> Connector_JST:JST_PH_B5B-PH-K_1x05_P2.00mm_Vertical; symbol Connector_Generic:Conn_01x04 -> Connector_Generic:Conn_01x05
- R205: value 10M -> 100k
- R208: value 1M -> 100k
Connections:
- net GND: now also C212.2, U204.2 (GND)
- net VBAT: now also J203.5 (Pin_5); no longer J203.4 (Pin_4)
- net VIN_LADER: now also U204.1 (IN)
- new net TMP_VCC: C212.1, J203.4 (Pin_4), U204.5 (OUT)
- no-connect marks 1 -> 3
Other:
- note added: "Laderegler BQ25185 (3.2/3.3): 4,1 V, 150 mA; CE und NTC von der Ladesperre der Akku-Platine; TMP_VCC nur bei Sonne"
- note removed: "Laderegler BQ25185 (3.2/3.3): 4,1 V, 150 mA, CE von der Ladesperre der Akku-Platine, NTC am TS"
- moved on the sheet: C202, C203, C207, C208, C209, C210, C211, R201, R202, R206, R207, R208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

Commit message: update
Parts:
- C204: value 10µ -> 22µ 25V X5R; footprint Capacitor_SMD:C_0805_2012Metric -> Capacitor_SMD:C_1206_3216Metric
- C208, C209: value 1µ -> 2,2µ 16V X7R
- C212: value 2,2µ -> 4,7µ 16V X7R; footprint Capacitor_SMD:C_0603_1608Metric -> Capacitor_SMD:C_0805_2012Metric
Other:
- note added: "1 Solar und USB → Schottky-Dioden → VIN_LADER (TVS, Messung der Eingangsspannung)"
- note added: "2 Laderegler BQ25185: 4,1 V, 150 mA; CE und TS kommen von der Ladesperre der Akku-Platine"
- note added: "3 Akku-Stecker J203, TMP_VCC"
- note added: "4 SYS → 3,3 V (RT9080) → geschaltete Sensorschiene 3V3_SW (TPS22917, Ein/Aus von der MCU)"
- note added: "J203: Kabel 1:1 zur Akku-Platine J1 (anschluesse.md). TMP_VCC aus dem TPS70933 am Ladereingang gibt es nur bei Sonne/USB; ohne TMP_VCC sperrt die Ladesperre (sicherheit-akku.md)."
- note removed: "3,3 V (RT9080, 3.6) und geschaltete Sensorschiene 3V3_SW (TPS22917, 3.7)"
- note removed: "Laderegler BQ25185 (3.2/3.3): 4,1 V, 150 mA; CE und NTC von der Ladesperre der Akku-Platine; TMP_VCC nur bei Sonne"
- note removed: "Solar-Eingang (versorgung.md 3.1): Schottky je Panel, TVS, Messung der Ladereingangsspannung"
- moved on the sheet: C201, C202, C203, C204, C205, C206, C207, C208, C209, C210, C211, C212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
