File: hardware/kicad/hauptplatine/versorgung.kicad_sch (KiCad schematic)
At the start: 34 parts, among them J201 Solar 1, J202 Solar 2, J203 Akku (JST PH 5), U201 BQ25185DLHR, U202 RT9080-33GJ5, U203 TPS22917DBV, U204 TPS70933DBV

Commit message: update
Footprints BQ25185, Ra-01SH, DEGSON 15EDGRC-3.5 (2-6P) in Bienen.pretty; HW-02 Akkuhalter Keystone 1042 SMD; SCH26-13 Klemmen einreihig mit LCSC-Nummern. Tests: ERC 0, Pin/Footprint 0 Abweichungen, Netzprüfung 178/178, alle_tests_linux.sh rc=0
Parts:
- J201, J202: footprint Connector_Phoenix_MC:PhoenixContact_MC_1,5_2-G-3.5_1x02_P3.50mm_Horizontal -> Bienen:DEGSON_15EDGRC-3.5-02P; LCSC (none) -> C5160225
Changed lines of the file:
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@@
 			)
 		)
-		(property "Footprint" "Connector_Phoenix_MC:PhoenixContact_MC_1,5_2-G-3.5_1x02_P3.50mm_Horizontal"
+		(property "Footprint" "Bienen:DEGSON_15EDGRC-3.5-02P"
 			(at 35.56 99.06 0)
 			(hide yes)
@@
 			)
 		)
+		(property "LCSC" "C5160225"
+			(at 35.56 99.06 0)
+			(hide yes)
+			(show_name no)
+			(do_not_autoplace no)
+			(effects
+				(font
+					(size 1.27 1.27)
+				)
+			)
+		)
 		(pin "1"
 		)
@@
 			)
 		)
-		(property "Footprint" "Connector_Phoenix_MC:PhoenixContact_MC_1,5_2-G-3.5_1x02_P3.50mm_Horizontal"
+		(property "Footprint" "Bienen:DEGSON_15EDGRC-3.5-02P"
 			(at 35.56 78.74 0)
 			(hide yes)
@@
 			)
 		)
-		(property "Description" "DEGSON 15EDGRHC-3.5 (Platzhalter-Footprint Phoenix MC 3,5 mm) [P]"
+		(property "Description" "DEGSON 15EDGRC-3.5-02P (einreihig, SCH26-13)"
 			(at 35.56 78.74 0)
 			(hide yes)
+			(show_name no)
+			(do_not_autoplace no)
+			(effects
+				(font
+					(size 1.27 1.27)
+				)
+			)
+		)
+		(property "LCSC" "C5160225"
+			(at 35.56 78.74 0)
+			(hide yes)

Commit message: update
"Hauptplatine grob platziert (platine_bestuecken.py, 139 Bauteile, Schaltplanabgleich 0); Gehäuse mit STEP geprüft: Lochbild bestätigt, Freiraum über Platine >= 44,3 mm (HW-03 erfüllt), Dombohrung Ø 2,4 mm korrigiert, Lichtleiter ca. 19,4 mm. Tests: ERC 0, Netzprüfung 178/178, alle_tests_linux.sh rc=0"
Parts:
- TP201, TP202: now left out of the parts list
Changed lines of the file:
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@@
 		(body_style 1)
 		(exclude_from_sim no)
-		(in_bom yes)
+		(in_bom no)
 		(on_board yes)
 		(in_pos_files yes)
@@
 		(body_style 1)
 		(exclude_from_sim no)
-		(in_bom yes)
-		(on_board yes)
-		(in_pos_files yes)
+		(in_bom no)
+		(on_board yes)
+		(in_pos_files yes)

Commit message: HW-06: Akku auf der Hauptplatine (Blatt Akku, Akku-Platine entfällt); HW-05: USB mit VBUS-Erkennung an PB13; Routing-Werkzeuge; Aufräumen: Restbezüge Akku-Platine, README-Stand; ERC 0, Netzprüfung 168/168, Pin/Footprint 0; Platine platziert, nicht geroutet
Parts:
- removed J203: Akku (JST PH 5), Connector_JST:JST_PH_B5B-PH-K_1x05_P2.00mm_Vertical, symbol Connector_Generic:Conn_01x05
Other:
- note added: "2 Laderegler BQ25185: 4,1 V, 150 mA; CE und TS kommen von der Ladesperre (Blatt Akku)"
- note added: "3 Zum Blatt Akku: VBAT, CE_LADEN, NTC, TMP_VCC"
- note added: "Zelle, Zellschutz und Ladesperre auf Blatt Akku (HW-06). TMP_VCC aus dem TPS70933 am Ladereingang gibt es nur bei Sonne/USB; ohne TMP_VCC sperrt die Ladesperre (sicherheit-akku.md)."
- note removed: "2 Laderegler BQ25185: 4,1 V, 150 mA; CE und TS kommen von der Ladesperre der Akku-Platine"
- note removed: "3 Akku-Stecker J203, TMP_VCC"
- note removed: "J203: Kabel 1:1 zur Akku-Platine J1 (anschluesse.md). TMP_VCC aus dem TPS70933 am Ladereingang gibt es nur bei Sonne/USB; ohne TMP_VCC sperrt die Ladesperre (sicherheit-akku.md)."
