File: hardware/kicad/hauptplatine/waage.kicad_sch (KiCad schematic)
At the start: 28 parts, among them J501 Wägezelle, Q501 S8550, U501 TPS61240DRVR, U502 HX711

Commit message: update
Parts:
- D501: footprint (none) -> Package_SON:USON-10_2.5x1.0mm_P0.5mm
- Q501: footprint (none) -> Package_TO_SOT_SMD:SOT-23
- U501: footprint (none) -> Package_SON:WSON-6-1EP_2x2mm_P0.65mm_EP1x1.6mm
- U502: footprint (none) -> Package_SO:SOIC-16_3.9x9.9mm_P1.27mm
Changed lines of the file:
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@@
 			)
 		)
-		(property "Footprint" ""
+		(property "Footprint" "Package_SON:WSON-6-1EP_2x2mm_P0.65mm_EP1x1.6mm"
 			(at 86.36 124.46 0)
 			(hide yes)
@@
 			)
 		)
-		(property "Footprint" ""
+		(property "Footprint" "Package_SON:USON-10_2.5x1.0mm_P0.5mm"
 			(at 78.74 215.9 0)
 			(hide yes)
@@
 			)
 		)
-		(property "Footprint" ""
+		(property "Footprint" "Package_TO_SOT_SMD:SOT-23"
 			(at 226.06 129.54 0)
 			(hide yes)
@@
 			)
 		)
-		(property "Footprint" ""
+		(property "Footprint" "Package_SO:SOIC-16_3.9x9.9mm_P1.27mm"
 			(at 264.16 157.48 0)
 			(hide yes)

Commit message: update
Footprints BQ25185, Ra-01SH, DEGSON 15EDGRC-3.5 (2-6P) in Bienen.pretty; HW-02 Akkuhalter Keystone 1042 SMD; SCH26-13 Klemmen einreihig mit LCSC-Nummern. Tests: ERC 0, Pin/Footprint 0 Abweichungen, Netzprüfung 178/178, alle_tests_linux.sh rc=0
Parts:
- J501: footprint Connector_Phoenix_MC:PhoenixContact_MC_1,5_5-G-3.5_1x05_P3.50mm_Horizontal -> Bienen:DEGSON_15EDGRC-3.5-05P; LCSC (none) -> C7603439
Changed lines of the file:
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@@
 			)
 		)
-		(property "Footprint" "Connector_Phoenix_MC:PhoenixContact_MC_1,5_5-G-3.5_1x05_P3.50mm_Horizontal"
+		(property "Footprint" "Bienen:DEGSON_15EDGRC-3.5-05P"
 			(at 45.72 177.8 0)
 			(hide yes)
@@
 			)
 		)
-		(property "Description" "= J4 in anschluesse.md: 1 Schirm, 2 E−, 3 S−, 4 S+, 5 E+; DEGSON 15EDGRHC-3.5 5-polig (Platzhalter Phoenix MC) [P]; Schirm nur hier an Masse"
+		(property "Description" "= J4 in anschluesse.md: 1 Schirm, 2 E−, 3 S−, 4 S+, 5 E+; DEGSON 15EDGRC-3.5-05P; Schirm nur hier an Masse"
 			(at 45.72 177.8 0)
 			(hide yes)
+			(show_name no)
+			(do_not_autoplace no)
+			(effects
+				(font
+					(size 1.27 1.27)
+				)
+			)
+		)
+		(property "LCSC" "C7603439"
+			(at 45.72 177.8 0)
+			(hide yes)
