File: hardware/kicad/hauptplatine/waage.kicad_sch (KiCad schematic)
At the start: 28 parts, among them J501 Wägezelle, Q501 S8550, U501 TPS61240DRVR, U502 HX711

Commit message: Review-Nachtrag: mikrofon.md J601 Pin 5/6 berichtigt, Q501 ohne unverifizierte LCSC-Nummer, R313 Entladung BLE_VCC
Netzpruefung 230/230, ERC 0, Pin/Footprint 186/0. PDF noch nicht neu erzeugt (Datei durch einen Viewer gesperrt).

Co-Authored-By: Claude Fable 5.1 <noreply@anthropic.com>
Parts:
- Q501: value S8550 -> S8550 (1 B, 2 E, 3 C); LCSC C397181 -> (none)
Changed lines of the file:
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@@
 			)
 		)
-		(property "Value" "S8550"
+		(property "Value" "S8550 (1 B, 2 E, 3 C)"
 			(at 222.52 131.14 0)
 			(show_name no)
@@
 			(at 226.06 129.54 0)
 			(hide yes)
-			(show_name no)
-			(do_not_autoplace no)
-			(effects
-				(font
-					(size 1.27 1.27)
-				)
-			)
-		)
-		(property "LCSC" "C397181"
-			(at 226.06 129.54 0)
-			(hide yes)
