File: hardware/kicad/hauptplatine/akku.kicad_sch (KiCad schematic)
At the start: 22 parts, among them J1 JST PH 5-polig, J2 Strommessung, Q1 FS8205, Q2 AO3400A, Q3 AO3400A, U1 HY2111-GB, U2 TMP390A2DRL, U3 TMP390A2DRL

Commit message: HW-06: Akku auf der Hauptplatine (Blatt Akku, Akku-Platine entfällt); HW-05: USB mit VBUS-Erkennung an PB13; Routing-Werkzeuge; Aufräumen: Restbezüge Akku-Platine, README-Stand; ERC 0, Netzprüfung 168/168, Pin/Footprint 0; Platine platziert, nicht geroutet
Parts:
- removed BT1: 18650 3,6 V, Battery:BatteryHolder_Keystone_1042_1x18650, symbol Device:Battery_Cell
- removed C1, C2, C3: 100n, Capacitor_SMD:C_0603_1608Metric, symbol Device:C
- removed J1: JST PH 5-polig, Connector_JST:JST_PH_S5B-PH-K_1x05_P2.00mm_Horizontal, symbol Connector_Generic:Conn_01x05
- removed J2: Strommessung, Connector_PinHeader_2.54mm:PinHeader_1x02_P2.54mm_Vertical, symbol Connector_Generic:Conn_01x02
- removed JP1: Messbrücke B+, Jumper:SolderJumper-2_P1.3mm_Bridged_RoundedPad1.0x1.5mm, symbol Jumper:SolderJumper_2_Bridged
- removed Q1: FS8205, Package_TO_SOT_SMD:SOT-23-6, symbol Bienen:FS8205
- removed Q2, Q3: AO3400A, Package_TO_SOT_SMD:SOT-23, symbol Transistor_FET:AO3400A
- removed R1: 100, Resistor_SMD:R_0603_1608Metric, symbol Device:R
- removed R2: 2k, Resistor_SMD:R_0603_1608Metric, symbol Device:R
- removed R3, R6: 2,49k 1%, Resistor_SMD:R_0603_1608Metric, symbol Device:R
- removed R4, R7: 18,7k 1%, Resistor_SMD:R_0603_1608Metric, symbol Device:R
- removed R5, R8: 100k, Resistor_SMD:R_0603_1608Metric, symbol Device:R
- removed TH1: 10k B3435, Resistor_SMD:R_0603_1608Metric, symbol Device:Thermistor_NTC
- removed U1: HY2111-GB, Package_TO_SOT_SMD:SOT-23-6, symbol Bienen:HY2111-GB
- removed U2, U3: TMP390A2DRL, Package_TO_SOT_SMD:SOT-563, symbol Bienen:TMP390
- added BT801: 18650 3,6 V, Battery:BatteryHolder_Keystone_1042_1x18650, symbol Device:Battery_Cell
- added C801, C802, C803: 100n, Capacitor_SMD:C_0603_1608Metric, symbol Device:C
- added J801: Strommessung, Connector_PinHeader_2.54mm:PinHeader_1x02_P2.54mm_Vertical, symbol Connector_Generic:Conn_01x02
- added JP801: Messbrücke B+, Jumper:SolderJumper-2_P1.3mm_Bridged_RoundedPad1.0x1.5mm, symbol Jumper:SolderJumper_2_Bridged
- added Q801: FS8205, Package_TO_SOT_SMD:SOT-23-6, symbol Bienen:FS8205
- added Q802, Q803: AO3400A, Package_TO_SOT_SMD:SOT-23, symbol Transistor_FET:AO3400A
- added R801: 100, Resistor_SMD:R_0603_1608Metric, symbol Device:R
- added R802: 2k, Resistor_SMD:R_0603_1608Metric, symbol Device:R
- added R803, R806: 2,49k 1%, Resistor_SMD:R_0603_1608Metric, symbol Device:R
- added R804, R807: 18,7k 1%, Resistor_SMD:R_0603_1608Metric, symbol Device:R
- added R805, R808: 100k, Resistor_SMD:R_0603_1608Metric, symbol Device:R
- added TH801: 10k B3435, Resistor_SMD:R_0603_1608Metric, symbol Device:Thermistor_NTC
- added U801: HY2111-GB, Package_TO_SOT_SMD:SOT-23-6, symbol Bienen:HY2111-GB
- added U802, U803: TMP390A2DRL, Package_TO_SOT_SMD:SOT-563, symbol Bienen:TMP390
Connections:
- net B+: now also BT801.1 (+), J801.1 (Pin_1), JP801.1 (A), R801.1
- net B-: now also BT801.2 (-), C801.2, Q801.1 (S1), U801.6 (VSS)
- net D12: now also Q801.2 (D12), Q801.5 (D12)
- net GATE_CE: now also Q802.1 (G), R805.2, U802.4 (~{OUTB}), U802.6 (~{OUTA})
- net GATE_ENTL: now also Q801.6 (G1), U801.1 (OD)
- net GATE_LADE: now also Q801.4 (G2), U801.3 (OC)
- net GATE_NTC: now also Q803.1 (G), R808.2, U803.6 (~{OUTA})
- net GND: now also C802.2, C803.2, Q801.3 (S2), Q802.2 (S), Q803.2 (S), R802.2, R803.2, R804.2, R806.2, R807.2, U802.3 (GND), U803.3 (GND)
- net HY_CS: now also R802.1, U801.2 (CS)
- net HY_VDD: now also C801.1, R801.2, U801.5 (VDD)
- net NTC: now also TH801.1
- net NTC_FUSS: now also Q803.3 (D), TH801.2
- net SETA1: now also R803.1, U802.1 (SETA)
- net SETA2: now also R806.1, U803.1 (SETA)
- net SETB1: now also R804.1, U802.2 (SETB)
- net SETB2: now also R807.1, U803.2 (SETB)
- net TMP_VCC: now also C802.1, C803.1, R805.1, R808.1, U802.5 (VDD), U803.5 (VDD)
- new net CE_LADEN: Q802.3 (D)
- new net VBAT: J801.2 (Pin_2), JP801.2 (B)
Other:
- note added: "1 Leistungspfad: Zelle → Messbrücke JP801 → VBAT (P+) zum Laderegler"
- note added: "2 Zellschutz im Minuspfad: HY2111 schaltet Q801 (M1 Entladen, M2 Laden); GND = P−, B− nur als Insel an der Zelle"
- note added: "3 Ladesperre Stufe 2 (SCH26-03): U803 öffnet über 42 °C mit Q803 den NTC-Kreis → TS offen → BQ25185 lädt nicht"
- note added: "TMP_VCC kommt vom TPS70933 am Ladereingang: nur bei Sonne/USB vorhanden; fehlt es, sperren beide Stufen. Keine Verbindung der Sperre zu B+/B− (SCH26-01). Layout: TH801, U802, U803 direkt unter der Zelle (Wärmeleitpad)."
- note added: "U802 sperrt außerhalb +5 … 42 °C über Q802: CE_LADEN high → BQ25185 lädt nicht"
- note removed: "1 Leistungspfad: Zelle → Messbrücke JP1 → P+ zum Stecker J1"
- note removed: "2 Zellschutz im Minuspfad: HY2111 schaltet Q1 (M1 Entladen, M2 Laden); GND = P−"
- note removed: "3 Ladesperre Stufe 2 (SCH26-03): U3 öffnet über 42 °C mit Q3 den NTC-Kreis → TS offen → BQ25185 lädt nicht"
- note removed: "TMP_VCC kommt von der Hauptplatine (TPS70933 am Ladereingang): nur bei Sonne/USB vorhanden. Fehlt es oder reißt eine Ader, sperren beide Stufen. Keine Verbindung der Sperre zu B+/B− (SCH26-01)."
- note removed: "U2 sperrt außerhalb +5 … 42 °C über Q2: CE_FREI high → BQ25185 lädt nicht"
- title: Akku-Platine: Zellschutz, Ladesperre -> Akku: Zelle 18650, Zellschutz, Temperatur-Ladesperre
