File: hardware/kicad/hauptplatine/mikrofon.kicad_sch (KiCad schematic)
At the start: 31 parts, among them J601 Mikrofone, U601 TLV320ADC3101IRGET, U602 TPS70918DBVR, U603 74LVC1G17GW

Commit message: HW-10: dritter Mikrofoneingang (Elektret 2 an IN2R/IN3R, Klemme J602 = J12 mit ESD D602); Pin-Review aller ICs
HW-10 (Philipp): alle drei Anschlussmoeglichkeiten des TLV320ADC3101 belegt, bis zu drei Mikrofone;
rechter Kanal je Messung PDM oder Elektret 2. Netzpruefung 236/236, ERC 0, Pin/Footprint 186/0.
Pin-Review: STM32F411 (ST open pin data), TPS22917 CT an VIN, TPS61240, TMP390, HY2111, FS8205,
AO3400A/AO3401A, 74LVC1G17, HX711 gelesen – keine Abweichung; pin_footprint.py auf [V].

Co-Authored-By: Claude Fable 5.1 <noreply@anthropic.com>
Parts:
- added C625, C626: 1µ X7R, Capacitor_SMD:C_0603_1608Metric, symbol Device:C
- added C627, C628: 100p C0G, Capacitor_SMD:C_0603_1608Metric, symbol Device:C
- added C629: 1µ, Capacitor_SMD:C_0603_1608Metric, symbol Device:C
- added D602: ESDS304DBVR, Package_TO_SOT_SMD:SOT-23-5, symbol Power_Protection:ESDS304
- added J602: Mikrofon 2 (Elektret), Bienen:DEGSON_15EDGRC-3.5-04P, symbol Connector_Generic:Conn_01x04
- added R614, R615: 1k, Resistor_SMD:R_0603_1608Metric, symbol Device:R
Connections:
- net GND: now also C627.2, C628.2, C629.2, D602.2 (A), J602.1 (Pin_1), R615.2
- net MIC2_INP: now reaches U601.12 (IN2R(P))
- net MIC2_INP: now also C625.2
- net MIC2_INN: now reaches U601.13 (IN3R(M))
- net MIC2_INN: now also C626.2
- net MICBIAS2: now reaches U601.14 (MICBIAS2)
- net MICBIAS2: now also C629.1, R614.1
- new net MIC2_N: C626.1, C628.1, D602.1 (K), J602.3 (Pin_3), R615.1
- new net MIC2_P: C625.1, C627.1, D602.3 (K), J602.4 (Pin_4), R614.2
Other:
- note added: "2 Audio-ADC TLV320ADC3101: links Elektret 1 (analog), rechts MEMS (PDM) oder Elektret 2 (analog, HW-10); I²S an I2S3, I²C 0x18"
- note added: "6 Klemme J602 (= J12, 4-polig): Elektret 2 pseudo-differenziell an IN2R(P)/IN3R(M), MICBIAS2 über 2 × 1 kΩ (HW-10)"
- note added: "ESD D601 direkt an J601, D602 direkt an J602"
- note added: "Firmware: 3V3_SW aus → I²S- und I²C-Pins hochohmig (keine Rückspeisung in U601); fS 24 576 Hz, AOSR 128, DMCLK 3,146 MHz; Messung ohne Funk und ohne 5-V-Wandler; rechter Kanal je Messung PDM oder Elektret 2 (mikrofon.md)."
- note removed: "2 Audio-ADC TLV320ADC3101: links Elektret (analog), rechts MEMS (PDM); I²S an I2S3, I²C 0x18"
- note removed: "ESD D601 direkt an J601"
- note removed: "Firmware: 3V3_SW aus → I²S- und I²C-Pins hochohmig (keine Rückspeisung in U601); fS 24 576 Hz, AOSR 128, DMCLK 3,146 MHz; Messung ohne Funk und ohne 5-V-Wandler (mikrofon.md)."
- title: Mikrofon: Audio-ADC TLV320ADC3101, Elektret (analog) + MEMS IM69D127 (PDM), I²S an I2S3 -> Mikrofon: Audio-ADC TLV320ADC3101, Elektret 1 + 2 (analog) + MEMS IM69D127 (PDM), I²S an I2S3
- moved on the sheet: D601

Commit message: HW-10: Zaehlung der Mikrofone (Philipp): J601 = Mikrofone 1 + 2, J602/J12 = Mikrofon 3; Netze MIC3_*
Co-Authored-By: Claude Fable 5.1 <noreply@anthropic.com>
Parts:
- J601: value Mikrofone -> Mikrofone 1 + 2
- J602: value Mikrofon 2 (Elektret) -> Mikrofon 3 (Elektret)
Connections:
- net MIC2_INN renamed MIC3_INN
- net MIC2_INP renamed MIC3_INP
- net MIC2_N renamed MIC3_N
- net MIC2_P renamed MIC3_P
Other:
- note added: "6 Klemme J602 (= J12, 4-polig): Mikrofon 3 (zweite Elektretkapsel) pseudo-differenziell an IN2R(P)/IN3R(M), MICBIAS2 über 2 × 1 kΩ (HW-10)"
- note removed: "6 Klemme J602 (= J12, 4-polig): Elektret 2 pseudo-differenziell an IN2R(P)/IN3R(M), MICBIAS2 über 2 × 1 kΩ (HW-10)"
Changed lines of the file:
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@@
 		)
 	)
-	(text "6  Klemme J602 (= J12, 4-polig): Elektret 2 pseudo-differenziell an IN2R(P)/IN3R(M), MICBIAS2 über 2 × 1 kΩ (HW-10)"
+	(text "1  Versorgung: 3V3_ANA (AVDD, Ferrit + 10 Ω), 1V8_ADC (DVDD, TPS70918), 3V3_MEMS (Ferrit, über das Kabel)"
 		(exclude_from_sim no)
-		(at 160.02 198.12 0)
+		(at 30.48 35.56 0)
 		(effects
 			(font
@@
 		)
 	)
-	(text "1  Versorgung: 3V3_ANA (AVDD, Ferrit + 10 Ω), 1V8_ADC (DVDD, TPS70918), 3V3_MEMS (Ferrit, über das Kabel)"
+	(text "Firmware: 3V3_SW aus → I²S- und I²C-Pins hochohmig (keine Rückspeisung in U601); fS 24 576 Hz, AOSR 128, DMCLK 3,146 MHz; Messung ohne Funk und ohne 5-V-Wandler; rechter Kanal je Messung PDM oder Elektret 2 (mikrofon.md)."
 		(exclude_from_sim no)
-		(at 30.48 35.56 0)
+		(at 30.48 269.24 0)
 		(effects
 			(font
-				(size 2 2)
+				(size 1.5 1.5)
 			)
 			(justify left bottom)
 		)
 	)
-	(text "Firmware: 3V3_SW aus → I²S- und I²C-Pins hochohmig (keine Rückspeisung in U601); fS 24 576 Hz, AOSR 128, DMCLK 3,146 MHz; Messung ohne Funk und ohne 5-V-Wandler; rechter Kanal je Messung PDM oder Elektret 2 (mikrofon.md)."
+	(text "6  Klemme J602 (= J12, 4-polig): Mikrofon 3 (zweite Elektretkapsel) pseudo-differenziell an IN2R(P)/IN3R(M), MICBIAS2 über 2 × 1 kΩ (HW-10)"
 		(exclude_from_sim no)
-		(at 30.48 269.24 0)
+		(at 160.02 198.12 0)
 		(effects
 			(font
-				(size 1.5 1.5)
+				(size 2 2)
 			)
 			(justify left bottom)
@@
 		)
 	)
-	(label "3V3_MEMS"
-		(at 198.12 55.88 270)
+	(label "MIC3_INP"
+		(at 193.04 147.32 180)
 		(effects
 			(font
@@
 		)
 	)
-	(label "MIC_INP"
-		(at 193.04 137.16 180)
+	(label "3V3_MEMS"
+		(at 198.12 55.88 270)
 		(effects
 			(font
@@
 		)
 	)
-	(label "PDM_CLK_BUF"
-		(at 88.9 187.96 0)
+	(label "MIC_INP"
+		(at 193.04 137.16 180)
 		(effects
 			(font
 				(size 1.27 1.27)
 			)
-			(justify left bottom)
+			(justify right bottom)
 		)
 	)
-	(label "MIC2_INP"
-		(at 254 208.28 0)
+	(label "PDM_CLK_BUF"
+		(at 88.9 187.96 0)
 		(effects
 			(font
@@
 		)
 	)
-	(label "MICBIAS"
-		(at 139.7 95.25 90)
+	(label "MIC3_INP"
+		(at 254 208.28 0)
 		(effects
 			(font
@@
 		)
 	)
-	(label "MIC2_INN"
-		(at 254 223.52 0)
+	(label "MICBIAS"
+		(at 139.7 95.25 90)
 		(effects
 			(font
@@
 		)
 	)
-	(label "MIC2_INP"
-		(at 193.04 147.32 180)
-		(effects
-			(font
-				(size 1.27 1.27)
-			)
-			(justify right bottom)
-		)
-	)
 	(label "1V8_ADC"
 		(at 147.32 45.72 0)
@@
 		)
 	)
-	(label "MIC2_INN"
-		(at 193.04 149.86 180)
-		(effects
-			(font
-				(size 1.27 1.27)
-			)
-			(justify right bottom)
-		)
-	)
 	(label "MIC_INN"
 		(at 127 106.68 0)
@@
 		)
 	)
+	(label "MIC3_N"
+		(at 187.96 223.52 0)
+		(effects
+			(font
+				(size 1.27 1.27)
+			)
+			(justify left bottom)
+		)
+	)
 	(label "3V3_ANA"
 		(at 96.52 52.07 270)
@@
 		)
 	)
+	(label "MIC3_INN"
+		(at 254 223.52 0)
+		(effects
+			(font
+				(size 1.27 1.27)
+			)
+			(justify left bottom)
+		)
+	)
 	(label "1V8_ADC"
 		(at 172.72 44.45 90)
@@
 		)
 	)
-	(label "PDM_DATA"
-		(at 127 172.72 0)
+	(label "MIC3_P"
+		(at 182.88 208.28 0)
 		(effects
 			(font
@@
 		)
 	)
-	(label "PDM_DATA_K"
-		(at 60.96 172.72 0)
+	(label "PDM_DATA"
+		(at 127 172.72 0)
 		(effects
 			(font
@@
 		)
 	)
-	(label "MIC2_N"
-		(at 187.96 223.52 0)
+	(label "PDM_DATA_K"
+		(at 60.96 172.72 0)
 		(effects
 			(font
@@
 		)
 	)
-	(label "MIC2_P"
-		(at 182.88 208.28 0)
+	(label "3V3_ANA"
+		(at 266.7 44.45 90)
 		(effects
 			(font
@@
 		)
 	)
-	(label "3V3_ANA"
-		(at 266.7 44.45 90)
+	(label "MIC3_N"
+		(at 233.68 236.22 90)
 		(effects
 			(font
@@
 		)
 	)
-	(label "MIC2_P"
-		(at 236.22 236.22 90)
+	(label "PDM_CLK_ADC"
+		(at 193.04 160.02 180)
 		(effects
 			(font
 				(size 1.27 1.27)
 			)
-			(justify left bottom)
+			(justify right bottom)
 		)
 	)
-	(label "PDM_CLK_ADC"
-		(at 193.04 160.02 180)
+	(label "MIC3_INN"
+		(at 193.04 149.86 180)
 		(effects
 			(font
@@
 		)
 	)
-	(label "MIC2_N"
-		(at 233.68 236.22 90)
-		(effects
-			(font
-				(size 1.27 1.27)
-			)
-			(justify left bottom)
-		)
-	)
 	(label "3V3_ANA"
 		(at 218.44 119.38 90)
@@
 		)
 	)
+	(label "MIC3_P"
+		(at 236.22 236.22 90)
+		(effects
+			(font
+				(size 1.27 1.27)
+			)
+			(justify left bottom)
+		)
+	)
 	(label "1V8_ADC"
 		(at 279.4 44.45 90)
@@
 			)
 		)
-		(property "Value" "Mikrofon 2 (Elektret)"
+		(property "Value" "Mikrofon 3 (Elektret)"
 			(at 162.83 218.77 0)
 			(show_name no)
@@
 			)
 		)
-		(property "Description" "= J12 (HW-10): 1 Schirm, 2 frei (Verwechslungsschutz), 3 MIC2−, 4 MIC2+; zweiadriges geschirmtes Kabel 0,5–1 m, Kapsel schwebend über dem Paar, Schirm nur hier an Masse; DEGSON 15EDGRC-3.5-04P"
+		(property "Description" "= J12 (HW-10): 1 Schirm, 2 frei (Verwechslungsschutz), 3 MIC3−, 4 MIC3+; zweiadriges geschirmtes Kabel 0,5–1 m, Kapsel schwebend über dem Paar, Schirm nur hier an Masse; DEGSON 15EDGRC-3.5-04P"
 			(at 165.1 218.44 0)
 			(hide yes)
@@
 			)
 		)
-		(property "Value" "Mikrofone"
+		(property "Value" "Mikrofone 1 + 2"
 			(at 29.48 141.3 0)
 			(show_name no)

Commit message: HW-10: Mikrofon 3 ueber J601 Pin 5/6 statt eigener Klemme (Philipp); J602 entfaellt, D602 an J601
Pins 5/6 der RJ45 waren Masse-Paarpartner von VDD und DATA; jetzt MIC3+/MIC3-. Regel: Mikrofon 3 nur
bei stehendem PDM-Takt messen. Netzpruefung 229/229, ERC 0, Pin/Footprint 185/0; Dokumente nachgezogen.

Co-Authored-By: Claude Fable 5.1 <noreply@anthropic.com>
Parts:
- removed J602: Mikrofon 3 (Elektret), Bienen:DEGSON_15EDGRC-3.5-04P, symbol Connector_Generic:Conn_01x04
- J601: value Mikrofone 1 + 2 -> Mikrofone 1–3
Connections:
- net GND: no longer J601.5, J601.6
- net MIC3_N: now also J601.6
- net MIC3_P: now also J601.5
- no-connect marks 7 -> 6
Other:
- note added: "3 RJ45-Buchse J601 (= J5): MIC−, MIC+ (Elektret 1), MIC3+/MIC3− (Pin 5/6, HW-10), VDD, DATA, CLK (Schmitt-Puffer)"
- note added: "6 Mikrofon 3 (zweite Elektretkapsel) an J601 Pin 5/6, pseudo-differenziell an IN2R(P)/IN3R(M), MICBIAS2 über 2 × 1 kΩ (HW-10)"
- note added: "ESD D601 und D602 direkt an J601"
- note removed: "3 RJ45-Buchse J601 (= J5): MIC−, MIC+ (Elektret, MICBIAS 2,5 V über 2 × 1 kΩ), VDD, DATA, CLK (Schmitt-Puffer)"
- note removed: "6 Klemme J602 (= J12, 4-polig): Mikrofon 3 (zweite Elektretkapsel) pseudo-differenziell an IN2R(P)/IN3R(M), MICBIAS2 über 2 × 1 kΩ (HW-10)"
- note removed: "ESD D601 direkt an J601, D602 direkt an J602"
- moved on the sheet: C625, C626, C627, C628, D602, R614, R615

Commit message: HW-10: J601-Pinreihenfolge (Philipp): 4 MIC3+, 5 MIC3-, 6 VDD - jedes Mikrofon auf eigenem T568B-Paar
Standardkabel/-stecker, kein Sonderloeten; PDM-Regel fuer Durchgang 2 nur noch Empfehlung.
netz_tests.py prueft die Paarzuordnung. Netzpruefung 231/231, ERC 0, Pin/Footprint 186/0; PDF neu.

Co-Authored-By: Claude Fable 5.1 <noreply@anthropic.com>
Connections:
- net 3V3_MEMS: now also J601.6; no longer J601.4
- net MIC3_N: now also J601.5; no longer J601.6
- net MIC3_P: now also J601.4; no longer J601.5
Other:
- note added: "3 RJ45-Buchse J601 (= J5): MIC−, MIC+ (Elektret 1, Paar 7/8), MIC3+/MIC3− (Paar 4/5, HW-10), VDD (Pin 6), DATA, CLK (Schmitt-Puffer)"
- note added: "6 Mikrofon 3 (zweite Elektretkapsel) an J601 Pin 4/5 (eigenes Paar), pseudo-differenziell an IN2R(P)/IN3R(M), MICBIAS2 über 2 × 1 kΩ (HW-10)"
- note removed: "3 RJ45-Buchse J601 (= J5): MIC−, MIC+ (Elektret 1), MIC3+/MIC3− (Pin 5/6, HW-10), VDD, DATA, CLK (Schmitt-Puffer)"
- note removed: "6 Mikrofon 3 (zweite Elektretkapsel) an J601 Pin 5/6, pseudo-differenziell an IN2R(P)/IN3R(M), MICBIAS2 über 2 × 1 kΩ (HW-10)"
Changed lines of the file:
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@@
 		)
 	)
-	(text "3  RJ45-Buchse J601 (= J5): MIC−, MIC+ (Elektret 1), MIC3+/MIC3− (Pin 5/6, HW-10), VDD, DATA, CLK (Schmitt-Puffer)"
+	(text "3  RJ45-Buchse J601 (= J5): MIC−, MIC+ (Elektret 1, Paar 7/8), MIC3+/MIC3− (Paar 4/5, HW-10), VDD (Pin 6), DATA, CLK (Schmitt-Puffer)"
 		(exclude_from_sim no)
 		(at 30.48 96.52 0)
@@
 		)
 	)
-	(text "6  Mikrofon 3 (zweite Elektretkapsel) an J601 Pin 5/6, pseudo-differenziell an IN2R(P)/IN3R(M), MICBIAS2 über 2 × 1 kΩ (HW-10)"
+	(text "6  Mikrofon 3 (zweite Elektretkapsel) an J601 Pin 4/5 (eigenes Paar), pseudo-differenziell an IN2R(P)/IN3R(M), MICBIAS2 über 2 × 1 kΩ (HW-10)"
 		(exclude_from_sim no)
 		(at 160.02 198.12 0)
@@
 	(wire
 		(pts
-			(xy 48.26 137.16) (xy 55.88 137.16)
+			(xy 48.26 139.7) (xy 55.88 139.7)
 		)
 		(stroke
@@
 	(wire
 		(pts
-			(xy 48.26 134.62) (xy 55.88 134.62)
+			(xy 48.26 137.16) (xy 55.88 137.16)
 		)
 		(stroke
@@
 	(wire
 		(pts
-			(xy 63.5 139.7) (xy 63.5 157.48)
+			(xy 63.5 134.62) (xy 63.5 157.48)
 		)
 		(stroke
@@
 	(wire
 		(pts
-			(xy 48.26 139.7) (xy 63.5 139.7)
+			(xy 48.26 134.62) (xy 63.5 134.62)
 		)
 		(stroke
@@
 	)
 	(label "MIC3_P"
-		(at 55.88 137.16 0)
+		(at 55.88 139.7 0)
 		(effects
 			(font
@@
 	)
 	(label "MIC3_N"
-		(at 55.88 134.62 0)
+		(at 55.88 137.16 0)
 		(effects
 			(font
@@
 			)
 		)
-		(property "Description" "= J5 in anschluesse.md: RJ45 geschirmt ohne Übertrager; Paare nach T568B: 1/2 GND+CLK, 3/6 DATA+MIC3−, 4/5 VDD+MIC3+, 7/8 MIC+/MIC− (Elektret am Rand, weit weg vom Takt); seit HW-10 Mikrofon 3 auf den Pins 5/6 (vorher Masse-Paarpartner) – Firmware misst Mikrofon 3 nur bei stehendem PDM-Takt; Schirm nur hier an Masse; Teil und LCSC-Nummer wählt der Layouter [P]; NICHT mit Netzwerk-/PoE-Geräten verbinden"
+		(property "Description" "= J5 in anschluesse.md: RJ45 geschirmt ohne Übertrager; Paare nach T568B: 1/2 GND+CLK, 3/6 DATA+VDD, 4/5 MIC3+/MIC3−, 7/8 MIC+/MIC− (jedes Mikrofon auf einem eigenen Paar, Elektrets am Rand, weit weg vom Takt; HW-10: Mikrofon 3 auf 4/5, VDD von 4 auf 6; VDD ist für DATA der Rückleiter, am Kopf 100 nF und hier C611); Schirm nur hier an Masse; Teil und LCSC-Nummer wählt der Layouter [P]; NICHT mit Netzwerk-/PoE-Geräten verbinden"
 			(at 38.1 139.7 0)
 			(hide yes)
@@
 			)
 		)
-		(property "Description" "direkt hinter J601 neben D601 (anschluesse.md 3): Pins 5/6 der Buchse; zwei Kanäle frei; LCSC [P]"
+		(property "Description" "direkt hinter J601 neben D601 (anschluesse.md 3): Paar 4/5 der Buchse; zwei Kanäle frei; LCSC [P]"
 			(at 60.96 243.84 0)
 			(hide yes)
