File: hardware/kicad/akku-platine/akku.kicad_sch (KiCad schematic)
At the start: 16 parts, among them J1 JST PH 4-polig, J2 Strommessung, Q1 FS8205, Q2 AO3400A, U1 HY2111-GB, U2 TMP390A2DRL

Commit message: Update Regelwerk
Parts:
- added C3: 100n, Capacitor_SMD:C_0603_1608Metric, symbol Device:C
- added Q3: AO3400A, Package_TO_SOT_SMD:SOT-23, symbol Transistor_FET:AO3400A
- added R6: 2,49k 1%, Resistor_SMD:R_0603_1608Metric, symbol Device:R
- added R7: 18,7k 1%, Resistor_SMD:R_0603_1608Metric, symbol Device:R
- added R8: 100k, Resistor_SMD:R_0603_1608Metric, symbol Device:R
- added U3: TMP390A2DRL, Package_TO_SOT_SMD:SOT-563, symbol Bienen:TMP390
- J1: value JST PH 4-polig -> JST PH 5-polig; footprint Connector_JST:JST_PH_S4B-PH-K_1x04_P2.00mm_Horizontal -> Connector_JST:JST_PH_S5B-PH-K_1x05_P2.00mm_Horizontal; symbol Connector_Generic:Conn_01x04 -> Connector_Generic:Conn_01x05
- R5: value 10M -> 100k
Connections:
- net GND: now also C3.2, Q3.2 (S), R6.2, R7.2, U3.3 (GND); no longer TH1.2
- net P+: now also J1.5 (Pin_5); no longer C2.1, J1.4 (Pin_4), R5.1, U2.5 (VDD)
- net SETA renamed SETA1
- net SETB renamed SETB1
- new net GATE_NTC: Q3.1 (G), R8.2, U3.6 (~{OUTA})
- new net NTC_FUSS: Q3.3 (D), TH1.2
- new net SETA2: R6.1, U3.1 (SETA)
- new net SETB2: R7.1, U3.2 (SETB)
- new net TMP_VCC: C2.1, C3.1, J1.4 (Pin_4), R5.1, R8.1, U2.5 (VDD), U3.5 (VDD)
- no-connect marks 1 -> 2
Other:
- note added: "Ladesperre Stufe 1: TMP390 U2 sperrt über CE außerhalb +5 … 42 °C"
- note added: "Ladesperre Stufe 2 (SCH26-03): TMP390 U3 öffnet mit Q3 den NTC-Kreis über 42 °C → BQ25185 sperrt (TS offen)"
- note added: "U2, U3 und TH1 direkt unter der Zelle (Wärmeleitpad). Leitungsbruch CE_FREI oder TMP_VCC → Laden gesperrt. Keine Verbindung von TMP_VCC/GATE_* zu B+/B− (kein Pfad am Zellschutz vorbei, SCH26-01)."
- note removed: "Ladesperre: TMP390 (Stufe 1, +5 … 42 °C) und NTC für BQ25185 (Stufe 2)"
- note removed: "TMP390 und NTC direkt unter der Zelle anordnen (Wärmekopplung). Leitungsbruch an CE_FREI: Pull-up auf der Hauptplatine → CE high → Laden gesperrt."
- moved on the sheet: C2, Q2, R3, R4, R5, TH1, U2

Commit message: update
Other:
- note added: "1 Leistungspfad: Zelle → Messbrücke JP1 → P+ zum Stecker J1"
- note added: "2 Zellschutz im Minuspfad: HY2111 schaltet Q1 (M1 Entladen, M2 Laden); GND = P−"
- note added: "3 Ladesperre Stufe 2 (SCH26-03): U3 öffnet über 42 °C mit Q3 den NTC-Kreis → TS offen → BQ25185 lädt nicht"
- note added: "4 Ladesperre Stufe 1 (CE)"
- note added: "TMP_VCC kommt von der Hauptplatine (TPS70933 am Ladereingang): nur bei Sonne/USB vorhanden. Fehlt es oder reißt eine Ader, sperren beide Stufen. Keine Verbindung der Sperre zu B+/B− (SCH26-01)."
- note added: "U2 sperrt außerhalb +5 … 42 °C über Q2: CE_FREI high → BQ25185 lädt nicht"
- note removed: "Ladesperre Stufe 1: TMP390 U2 sperrt über CE außerhalb +5 … 42 °C"
- note removed: "Ladesperre Stufe 2 (SCH26-03): TMP390 U3 öffnet mit Q3 den NTC-Kreis über 42 °C → BQ25185 sperrt (TS offen)"
- note removed: "Quellen: HYCON HY2111 (LCSC C82747) Abschnitt 7/10; FS8205 (LCSC C32254); TI TMP390 SBOS904A Tab. 7-1/7-2; versorgung.md 3.3/3.4."
- note removed: "U2, U3 und TH1 direkt unter der Zelle (Wärmeleitpad). Leitungsbruch CE_FREI oder TMP_VCC → Laden gesperrt. Keine Verbindung von TMP_VCC/GATE_* zu B+/B− (kein Pfad am Zellschutz vorbei, SCH26-01)."
- note removed: "Zelle, Messbrücke, Stecker zur Hauptplatine"
- note removed: "Zellschutz: HY2111-GB + FS8205 (2,90 V aus, Freigabe durch Laden)"
- moved on the sheet: BT1, C1, C2, C3, J1, J2, JP1, Q1, Q2, Q3, R1, R2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

Commit message: Wetter-Eingang hinzugefügt
Changed lines of the file:
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@@
 					(size 1.27 1.27)
 				)
-				(justify right)
+				(justify left)
 			)
 		)
@@
 					(size 1.27 1.27)
 				)
-				(justify right)
+				(justify left)
 			)
 		)
