File: hardware/kicad/akku-platine/akku.kicad_sch (KiCad schematic)
At the start: 22 parts, among them J1 JST PH 5-polig, J2 Strommessung, Q1 FS8205, Q2 AO3400A, Q3 AO3400A, U1 HY2111-GB, U2 TMP390A2DRL, U3 TMP390A2DRL

Commit message: update
"Hauptplatine grob platziert (platine_bestuecken.py, 139 Bauteile, Schaltplanabgleich 0); Gehäuse mit STEP geprüft: Lochbild bestätigt, Freiraum über Platine >= 44,3 mm (HW-03 erfüllt), Dombohrung Ø 2,4 mm korrigiert, Lichtleiter ca. 19,4 mm. Tests: ERC 0, Netzprüfung 178/178, alle_tests_linux.sh rc=0"
Parts:
- JP1: now left out of the parts list
Changed lines of the file:
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@@
 		(body_style 1)
 		(exclude_from_sim no)
-		(in_bom yes)
+		(in_bom no)
 		(on_board yes)
 		(in_pos_files yes)
